File: AI.zero.template.kicad_pcb (KiCad board)
At the start: 2 copper layers, 65 x 30 mm, 8 parts

Commit message: Added text labels for the Phones connector
Other:
- board text added: "S"
- board text added: "T"

Commit message: bumped version to v1.1
Other:
- board text added: "AudioInjector.net Zero Template v1.1"
- board text removed: "AudioInjector.net Zero Template v1.0"
Changed lines of the file:
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@@
     (visible_elements FFFEFF7F)
     (pcbplotparams
-      (layerselection 0x010ff_80000001)
+      (layerselection 0x010ff_ffffffff)
       (usegerberextensions true)
       (usegerberattributes true)
@@
       (drillshape 0)
       (scaleselection 1)
-      (outputdirectory "flax.project21/"))
+      (outputdirectory "gerbers/"))
   )
   (net 0 "")
@@
     (effects (font (size 1 1) (thickness 0.25)))
   )
-  (gr_text "AudioInjector.net\nZero Template\nv1.0\n" (at 136.9 102.7) (layer F.SilkS)
+  (gr_text "AudioInjector.net\nZero Template\nv1.1\n" (at 136.9 102.7) (layer F.SilkS)
     (effects (font (size 1.5 1.5) (thickness 0.3)))
   )
